File: V1/ESP-relay_6ch-V1.kicad_pcb (KiCad board)
At the start: 2 copper layers, 173 x 67.8 mm, 91 parts, among them J1 24VDC, J2 24V INPUTS, J3 OUT1, J4 OUT1, J5 OUT1, J6 OUT1, J7 OUT1, J8 OUT1, K1 G5PZ-1A, K2 G5PZ-1A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

Commit message: updates
Other:
- net class Default removed
