File: V2/ESP-relay-6ch-V2.kicad_sch (KiCad schematic)
At the start: 109 parts

Commit message: update schematics title block
Parts:
- C1: value (none) -> 47uF/35V/6,3x5,4; footprint (none) -> Tales:CP_Elec_6.3x5.4
- C2: value (none) -> 0,33uF/35V; footprint (none) -> Tales:CP_EIA-3216-18_Kemet-A_Pad1.58x1.35mm_HandSolder
- C3: value (none) -> 0,1uF/50V/0805; footprint (none) -> Tales:C_0805_2012Metric
- C4, C5, C6, C7, C8, C9: value (none) -> 33nF/50V/0805; footprint (none) -> Tales:C_0805_2012Metric
- D1: value (none) -> SM4007PL/SOD-123; footprint (none) -> Tales:D_SOD-123
- D10, D5, D6, D7, D8, D9: value (none) -> 9V1/500mW; footprint (none) -> Tales:D_MiniMELF
- D11, D13, D15, D17, D19, D21: value (none) -> BLUE/0603; footprint (none) -> Tales:LED_0603_1608Metric
- D12, D14, D16, D18, D20, D22: value (none) -> 1N4148/SOD-123; footprint (none) -> Tales:D_SOD-123
- D2, D3, D4: value (none) -> GREEN/0603; footprint (none) -> Tales:LED_0603_1608Metric
- D23, D24: value (none) -> 7V5/5W/SMB; footprint (none) -> Tales:D_SMB
- J1: value (none) -> POWER & INPUTS; footprint (none) -> Tales:TerminalBlock_Phoenix_MKDS-3-8-5.08_1x08_P5.08mm_Horizontal
- J2, J3, J4, J5, J6, J7: value (none) -> OUT1; footprint (none) -> Tales:TerminalBlock_Phoenix_MKDS-3-2-5.08_1x02_P5.08mm_Horizontal
- K1, K2, K3, K4, K5, K6: value (none) -> G5PZ-1A; footprint (none) -> Tales:Relay_SPST_Omron-G5PZ-1A
- Q1, Q2, Q3, Q4, Q5, Q6: value (none) -> MMBT2222A/SOT-23-3; footprint (none) -> Tales:SOT-23
- R1: value (none) -> 270R/0,125W/0805; footprint (none) -> Tales:R_0805_2012Metric
- R10, R12, R14, R4, R6, R8: value (none) -> 1k2/0,125W/0805; footprint (none) -> Tales:R_0805_2012Metric
- R11, R13, R15, R5, R7, R9: value (none) -> 3k3/0,125W/0805; footprint (none) -> Tales:R_0805_2012Metric
- R16, R18, R20, R22, R24, R26: value (none) -> 1k/0,125W/0805; footprint (none) -> Tales:R_0805_2012Metric
- R17, R19, R21, R23, R25, R27, R42: value (none) -> 4k7/0,125W/0805; footprint (none) -> Tales:R_0805_2012Metric
- R2: value (none) -> 3k9/0,125W/0805; footprint (none) -> Tales:R_0805_2012Metric
- R28, R29, R30, R31, R32, R33, R34, R35: value (none) -> 56R/0,125W/0805; footprint (none) -> Tales:R_0805_2012Metric
- R3: value (none) -> 680R/0,125W/0805; footprint (none) -> Tales:R_0805_2012Metric
- R36, R37, R38, R39, R40, R41: value (none) -> 10k/0,125W/0805; footprint (none) -> Tales:R_0805_2012Metric
- RV1, RV2, RV3, RV4, RV5, RV6: value (none) -> 250VAC; footprint (none) -> Tales:RV_Disc_D12mm_W3.9mm_P7.5mm
- U1: value (none) -> L78M05/TO-252-2; footprint (none) -> Tales:TO-252-2
- U2: value (none) -> Olimex_ESP32-POE; footprint (none) -> Tales:Olimex_ESP32-POE_Pads
- U3: value (none) -> WeMos_D1_mini; footprint (none) -> Tales:WEMOS_D1_mini_light_pads
- U4, U5, U6, U7, U8, U9: value (none) -> LTV-817S; footprint (none) -> Tales:SMDIP-4_W9.53mm
Other:
- title: ESP 6 Relay Module -> ESP 6x 24VDC Input 6x Relay Output Module
